File: GyroDrive-Commutator-Adaptor.brd (EAGLE design)
At the start: 108 x 76.2 mm, 26 parts, among them U1 HALL, U2 PCA9517, U3 5V, U4 2.5V, U5 INA2141U, U6 INA2141U, U7 INA2141U, X1 NORCOMP-DB25-SMD-MALE

Commit message: Added more bypass capacitors (one for each power supply on each instrumentation amp)
Parts:
- added C10, C7, C8, C9: 100nF, resistor:C0805
Connections:
- net AGND: now also C10.2, C7.2, C8.2, C9.2
- net V+: now also C7.1, C9.1
- net V-: now also C10.1, C8.1
Routing:
- net AGND: track 99.9 -> 107.0 mm, vias 14 -> 17
- net CHAN4: track 21.2 -> 15.7 mm
- net V+: track 185.7 -> 189.9 mm
- net V-: track 75.3 -> 78.0 mm
- net ICOM: track 29.2 -> 30.6 mm
